Commit message: Use the local robotiq_description instead of the /opt/ros one

File: src/ros_robotiq_description/ros_robotiq_description/urdf/moveit_urdf.urdf (robot description, URDF)
Before this commit: robot ur3_robotiq, 24 links, 23 joints
Links:
- link robotiq_85_base_link: geometry collision mesh filename=package://robotiq_description/meshes/collision/robotiq_base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; visual mesh filename=package://robotiq_description/meshes/visual/robotiq_base.dae
- link robotiq_85_left_finger_link: geometry collision mesh filename=package://robotiq_description/meshes/collision/left_finger.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; visual mesh filename=package://robotiq_description/meshes/visual/left_finger.dae
- link robotiq_85_left_finger_tip_link: geometry collision mesh filename=package://robotiq_description/meshes/collision/left_finger_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; visual mesh filename=package://robotiq_description/meshes/visual/left_finger_tip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
- link robotiq_85_left_inner_knuckle_link: geometry collision mesh filename=package://robotiq_description/meshes/collision/left_inner_k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; visual mesh filename=package://robotiq_description/meshes/visual/left_inner_knuc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
- link robotiq_85_left_knuckle_link: geometry collision mesh filename=package://robotiq_description/meshes/collision/left_knuckle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; visual mesh filename=package://robotiq_description/meshes/visual/left_knuckle.dae
- link robotiq_85_right_finger_link: geometry collision mesh filename=package://robotiq_description/meshes/collision/right_finger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; visual mesh filename=package://robotiq_description/meshes/visual/right_finger.dae
- link robotiq_85_right_finger_tip_link: geometry collision mesh filename=package://robotiq_description/meshes/collision/right_finger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; visual mesh filename=package://robotiq_description/meshes/visual/right_finger_ti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
- link robotiq_85_right_inner_knuckle_link: geometry collision mesh filename=package://robotiq_description/meshes/collision/right_inner_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; visual mesh filename=package://robotiq_description/meshes/visual/right_inner_knu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
- link robotiq_85_right_knuckle_link: geometry collision mesh filename=package://robotiq_description/meshes/collision/right_knuckl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; visual mesh filename=package://robotiq_description/meshes/visual/right_knuckle.d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

File: src/ros_robotiq_description/ros_robotiq_description/urdf/ur3e.urdf (robot description, URDF)
Before this commit: robot ur3_robotiq, 24 links, 23 joints
Links:
- link robotiq_85_base_link: geometry collision mesh filename=package://robotiq_description/meshes/collision/robotiq_base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; visual mesh filename=package://robotiq_description/meshes/visual/robotiq_base.dae
- link robotiq_85_left_finger_link: geometry collision mesh filename=package://robotiq_description/meshes/collision/left_finger.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; visual mesh filename=package://robotiq_description/meshes/visual/left_finger.dae
- link robotiq_85_left_finger_tip_link: geometry collision mesh filename=package://robotiq_description/meshes/collision/left_finger_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; visual mesh filename=package://robotiq_description/meshes/visual/left_finger_tip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
- link robotiq_85_left_inner_knuckle_link: geometry collision mesh filename=package://robotiq_description/meshes/collision/left_inner_k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; visual mesh filename=package://robotiq_description/meshes/visual/left_inner_knuc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
- link robotiq_85_left_knuckle_link: geometry collision mesh filename=package://robotiq_description/meshes/collision/left_knuckle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; visual mesh filename=package://robotiq_description/meshes/visual/left_knuckle.dae
- link robotiq_85_right_finger_link: geometry collision mesh filename=package://robotiq_description/meshes/collision/right_finger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; visual mesh filename=package://robotiq_description/meshes/visual/right_finger.dae
- link robotiq_85_right_finger_tip_link: geometry collision mesh filename=package://robotiq_description/meshes/collision/right_finger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; visual mesh filename=package://robotiq_description/meshes/visual/right_finger_ti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
- link robotiq_85_right_inner_knuckle_link: geometry collision mesh filename=package://robotiq_description/meshes/collision/right_inner_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; visual mesh filename=package://robotiq_description/meshes/visual/right_inner_knu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
- link robotiq_85_right_knuckle_link: geometry collision mesh filename=package://robotiq_description/meshes/collision/right_knuckl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; visual mesh filename=package://robotiq_description/meshes/visual/right_knuckle.d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
