Commit message: setup main xacro for the custom gripper

File: src/ros_robotiq_description/ros_robotiq_description/urdf/ur3e_robotiq.urdf.xacro (robot description, xacro)
@@ -10,5 +10,5 @@
   <!-- import end effector -->
   <xacro:include filename="$(find robotiq_description)/urdf/robotiq_2f_85_macro.urdf.xacro" />
-  <!-- import dapter macro -->
+  <!-- import adapter macro -->
   <xacro:include filename="$(find robotiq_description)/urdf/ur_to_robotiq_adapter.urdf.xacro" />
   <!-- import oakd_pro camera macros -->
@@ -29,4 +29,5 @@
   <xacro:arg name="safety_k_position" default="20"/>
   <xacro:arg name="mock_sensor_commands" default="false" />
+  <xacro:arg name="gripper_type" default="robotiq" />
   <!-- robotiq parameters -->
   <xacro:arg name="prefix" default="" />
@@ -65,23 +66,7 @@
   <!-- we have to force include_ros2_control to be false because the -->
   <!-- robotiq package violates some jazzy+ specific rules, the fixed control is below-->
-  <xacro:robotiq_gripper
-    name="$(arg name)"
-    prefix="$(arg prefix)"
-    parent="$(arg prefix)gripper_mount_link"
-    sim_ignition="$(arg sim_ignition)"
-    sim_isaac="$(arg sim_isaac)"
-    use_fake_hardware="$(arg use_fake_hardware)"
-    fake_sensor_commands="$(arg fake_sensor_commands)"
-    include_ros2_control="false"
-    com_port="$(arg com_port)"
-    >
-    <origin xyz="0 0 0" rpy="0 0 0" />          <!-- position robot in the world -->
-  </xacro:robotiq_gripper>
-  <!-- gripper to arm adapter -->
-  <xacro:ur_to_robotiq
-    prefix="$(arg prefix)"
-    connected_to="$(arg tf_prefix)tool0"
-    rotation="0.0"
-    />
+  <xacro:if value="${'$(arg gripper_type)' == 'custom'}">
+    <!-- We'll put the gripper stuff here once I export it -->
+  </xacro:if>
   <!-- wrist mounted OAK-D Pro camera -->
   <xacro:if value="$(arg use_oakd_pro)">
@@ -122,42 +107,63 @@
       </ros2_control>
     </xacro:macro>
-  <!-- Add fixed control for gripper -->
-  <ros2_control name="robotiq_gripper_system" type="system">
-    <hardware>
-      <!-- <plugin>mock_components/GenericSystem</plugin> -->
-      <plugin>gz_ros2_control/GazeboSimSystem</plugin>
-      <param name="fake_sensor_commands">True</param>
-      <param name="state_following_offset">0.0</param>
-    </hardware>
-    <!-- Main joint -->
-    <joint name="robotiq_85_left_knuckle_joint">
-      <command_interface name="position"/>
-      <state_interface name="position">
-        <param name="initial_value">0.7929</param>
-      </state_interface>
-      <state_interface name="velocity"/>
-    </joint>
-    <!-- Mimic joints-->
-    <joint name="robotiq_85_right_knuckle_joint">
-      <state_interface name="position"/>
-      <state_interface name="velocity"/>
-    </joint>
-    <joint name="robotiq_85_left_inner_knuckle_joint">
-      <state_interface name="position"/>
-      <state_interface name="velocity"/>
-    </joint>
-    <joint name="robotiq_85_right_inner_knuckle_joint">
-      <state_interface name="position"/>
-      <state_interface name="velocity"/>
-    </joint>
-    <joint name="robotiq_85_left_finger_tip_joint">
-      <state_interface name="position"/>
-      <state_interface name="velocity"/>
-    </joint>
-    <joint name="robotiq_85_right_finger_tip_joint">
-      <state_interface name="position"/>
-      <state_interface name="velocity"/>
-    </joint>
-  </ros2_control>
+  <xacro:if value="${'$(arg gripper_type)' == 'robotiq'}">
+    <xacro:robotiq_gripper
+      name="$(arg name)"
+      prefix="$(arg prefix)"
+      parent="$(arg prefix)gripper_mount_link"
+      sim_ignition="$(arg sim_ignition)"
+      sim_isaac="$(arg sim_isaac)"
+      use_fake_hardware="$(arg use_fake_hardware)"
+      fake_sensor_commands="$(arg fake_sensor_commands)"
+      include_ros2_control="false"
+      com_port="$(arg com_port)"
+      >
+      <origin xyz="0 0 0" rpy="0 0 0" />          <!-- position robot in the world -->
+    </xacro:robotiq_gripper>
+    <!-- gripper to arm adapter -->
+    <xacro:ur_to_robotiq
+      prefix="$(arg prefix)"
+      connected_to="$(arg tf_prefix)tool0"
+      rotation="0.0"
+      />
+    <!-- Add fixed control for gripper -->
+    <ros2_control name="robotiq_gripper_system" type="system">
+      <hardware>
+        <!-- <plugin>mock_components/GenericSystem</plugin> -->
+        <plugin>gz_ros2_control/GazeboSimSystem</plugin>
+        <param name="fake_sensor_commands">True</param>
+        <param name="state_following_offset">0.0</param>
+      </hardware>
+      <!-- Main joint -->
+      <joint name="robotiq_85_left_knuckle_joint">
+        <command_interface name="position"/>
+        <state_interface name="position">
+          <param name="initial_value">0.7929</param>
+        </state_interface>
+        <state_interface name="velocity"/>
+      </joint>
+      <!-- Mimic joints-->
+      <joint name="robotiq_85_right_knuckle_joint">
+        <state_interface name="position"/>
+        <state_interface name="velocity"/>
+      </joint>
+      <joint name="robotiq_85_left_inner_knuckle_joint">
+        <state_interface name="position"/>
+        <state_interface name="velocity"/>
+      </joint>
+      <joint name="robotiq_85_right_inner_knuckle_joint">
+        <state_interface name="position"/>
+        <state_interface name="velocity"/>
+      </joint>
+      <joint name="robotiq_85_left_finger_tip_joint">
+        <state_interface name="position"/>
+        <state_interface name="velocity"/>
+      </joint>
+      <joint name="robotiq_85_right_finger_tip_joint">
+        <state_interface name="position"/>
+        <state_interface name="velocity"/>
+      </joint>
+    </ros2_control>
+  </xacro:if>
   <!-- ros2 control instance -->
   <xacro:ur_ros2_control
@@ -170,6 +176,11 @@
   <gazebo>
     <plugin filename="libgz_ros2_control-system.so"
-            name="gz_ros2_control::GazeboSimROS2ControlPlugin">
-      <parameters>$(find ros_robotiq_description)/config/ur3e_robotiq_controllers.yaml</parameters>
+      name="gz_ros2_control::GazeboSimROS2ControlPlugin">
+      <xacro:if value="${'$(arg gripper_type)' == 'robotiq'}">
+        <parameters>$(find ros_robotiq_description)/config/ur3e_robotiq_controllers.yaml</parameters>
+      </xacro:if>
+      <xacro:if value="${'$(arg gripper_type)' == 'custom'}">
+        <!-- We'll put the gripper control stuff here once I export it -->
+      </xacro:if>
     </plugin>
   </gazebo>

Commit message: integrate custom gripper into launch files

File: src/ros_robotiq_description/ros_robotiq_description/urdf/ur3e_robotiq.urdf.xacro (robot description, xacro)
@@ -8,8 +8,11 @@
   <xacro:include filename="$(find ur_description)/urdf/inc/ur_sensors.xacro" />
   <!--<xacro:include filename="$(find ur_description)/urdf/ros2_control_mock_hardware.xacro" />  This doesnt work with gazebo -->
-  <!-- import end effector -->
-  <xacro:include filename="$(find robotiq_description)/urdf/robotiq_2f_85_macro.urdf.xacro" />
-  <!-- import adapter macro -->
-  <xacro:include filename="$(find robotiq_description)/urdf/ur_to_robotiq_adapter.urdf.xacro" />
+  <xacro:arg name="gripper_type" default="custom" />
+  <xacro:if value="${'$(arg gripper_type)' == 'robotiq'}">
+    <!-- import end effector -->
+    <xacro:include filename="$(find robotiq_description)/urdf/robotiq_2f_85_macro.urdf.xacro" />
+    <!-- import adapter macro -->
+    <xacro:include filename="$(find robotiq_description)/urdf/ur_to_robotiq_adapter.urdf.xacro" />
+   </xacro:if>
   <!-- import oakd_pro camera macros -->
   <xacro:include filename="$(find oakd_description)/urdf/oakd_pro.urdf.xacro" />
@@ -20,5 +23,4 @@
   <xacro:arg name="tf_prefix" default="" />
   <xacro:arg name="joint_limit_params" default="$(find ur3e_moveit_config)/config/joint_limits.yaml"/>
-  <!--<xacro:arg name="joint_limit_params" default="$(find ur_description)/config/$(arg ur_type)/joint_limits.yaml"/> -->
   <xacro:arg name="kinematics_params" default="$(find ur_description)/config/$(arg ur_type)/default_kinematics.yaml"/>
   <xacro:arg name="physical_params" default="$(find ur_description)/config/$(arg ur_type)/physical_parameters.yaml"/>
@@ -29,5 +31,4 @@
   <xacro:arg name="safety_k_position" default="20"/>
   <xacro:arg name="mock_sensor_commands" default="false" />
-  <xacro:arg name="gripper_type" default="robotiq" />
   <!-- robotiq parameters -->
   <xacro:arg name="prefix" default="" />
@@ -67,5 +68,11 @@
   <!-- robotiq package violates some jazzy+ specific rules, the fixed control is below-->
   <xacro:if value="${'$(arg gripper_type)' == 'custom'}">
-    <!-- We'll put the gripper stuff here once I export it -->
+    <xacro:include filename="$(find gripper_description)/urdf/colman-gripper.xacro"/>
+    <xacro:colman-gripper prefix="$(arg prefix)" include_gazebo_plugin="false"/>
+    <joint name="$(arg prefix)gripper_mount_joint" type="fixed">
+      <parent link="$(arg tf_prefix)tool0"/>
+      <child link="$(arg prefix)gripper_base"/>
+      <origin xyz="0 0 0" rpy="1.5708 0 0"/>
+    </joint>
   </xacro:if>
   <!-- wrist mounted OAK-D Pro camera -->
@@ -132,5 +139,5 @@
         <!-- <plugin>mock_components/GenericSystem</plugin> -->
         <plugin>gz_ros2_control/GazeboSimSystem</plugin>
-        <param name="fake_sensor_commands">True</param>
+        <param name="fake_sensor_commands">true</param>
         <param name="state_following_offset">0.0</param>
       </hardware>
@@ -181,5 +188,5 @@
       </xacro:if>
       <xacro:if value="${'$(arg gripper_type)' == 'custom'}">
-        <!-- We'll put the gripper control stuff here once I export it -->
+        <parameters>$(find ros_robotiq_description)/config/ur3e_gripper_controllers.yaml</parameters>
       </xacro:if>
     </plugin>
