Commit message: regenerate moveit config through setup wizard

File: src/ur3e_moveit_config/config/ur3_robotiq.ros2_control.xacro (robot description, xacro)
@@ -49,8 +49,8 @@
                 <state_interface name="velocity"/>
             </joint>
-            <joint name="robotiq_85_left_knuckle_joint">
+            <joint name="servotodrivegear">
                 <command_interface name="position"/>
                 <state_interface name="position">
-                  <param name="initial_value">${initial_positions['robotiq_85_left_knuckle_joint']}</param>
+                  <param name="initial_value">${initial_positions['servotodrivegear']}</param>
                 </state_interface>
                 <state_interface name="velocity"/>
