Commit message: add color to gripper in rviz and gazebo

File: src/gripper_description/gripper_description/urdf/colman-gripper.xacro (robot description, xacro)
@@ -5,4 +5,7 @@
     <xacro:property name="inertials_file" value="${xacro.load_yaml('$(find gripper_description)/config/inertials.yaml')}"/>
     <xacro:property name="inertials" value="${inertials_file['inertials']}"/>
+    <material name="gripper_dark_grey">
+      <color rgba="0.2 0.2 0.2 1.0"/>
+    </material>
     <link name="${prefix}gripper_base">
       <inertial>
@@ -16,4 +19,5 @@
           <mesh filename="package://gripper_description/meshes/visual/base.${visual_mesh_ext}" scale="0.001 0.001 0.001"/>
         </geometry>
+        <material name="gripper_dark_grey"/>
       </visual>
       <collision>
@@ -35,4 +39,5 @@
           <mesh filename="package://gripper_description/meshes/visual/left_gear.${visual_mesh_ext}" scale="0.001 0.001 0.001"/>
         </geometry>
+        <material name="gripper_dark_grey"/>
       </visual>
       <collision>
@@ -54,4 +59,5 @@
           <mesh filename="package://gripper_description/meshes/visual/right_gear.${visual_mesh_ext}" scale="0.001 0.001 0.001"/>
         </geometry>
+        <material name="gripper_dark_grey"/>
       </visual>
       <collision>
@@ -73,4 +79,5 @@
           <mesh filename="package://gripper_description/meshes/visual/left_arm_bottom.${visual_mesh_ext}" scale="0.001 0.001 0.001"/>
         </geometry>
+        <material name="gripper_dark_grey"/>
       </visual>
       <collision>
@@ -92,4 +99,5 @@
           <mesh filename="package://gripper_description/meshes/visual/right_arm_bottom.${visual_mesh_ext}" scale="0.001 0.001 0.001"/>
         </geometry>
+        <material name="gripper_dark_grey"/>
       </visual>
       <collision>
@@ -111,4 +119,5 @@
           <mesh filename="package://gripper_description/meshes/visual/bottom_stick_left.${visual_mesh_ext}" scale="0.001 0.001 0.001"/>
         </geometry>
+        <material name="gripper_dark_grey"/>
       </visual>
       <collision>
@@ -130,4 +139,5 @@
           <mesh filename="package://gripper_description/meshes/visual/bottom_stick_right.${visual_mesh_ext}" scale="0.001 0.001 0.001"/>
         </geometry>
+        <material name="gripper_dark_grey"/>
       </visual>
       <collision>
@@ -149,4 +159,5 @@
           <mesh filename="package://gripper_description/meshes/visual/top_stick_left.${visual_mesh_ext}" scale="0.001 0.001 0.001"/>
         </geometry>
+        <material name="gripper_dark_grey"/>
       </visual>
       <collision>
@@ -168,4 +179,5 @@
           <mesh filename="package://gripper_description/meshes/visual/top_stick_right.${visual_mesh_ext}" scale="0.001 0.001 0.001"/>
         </geometry>
+        <material name="gripper_dark_grey"/>
       </visual>
       <collision>
@@ -187,4 +199,5 @@
           <mesh filename="package://gripper_description/meshes/visual/drive_gear.${visual_mesh_ext}" scale="0.001 0.001 0.001"/>
         </geometry>
+        <material name="gripper_dark_grey"/>
       </visual>
       <collision>
@@ -275,4 +288,35 @@
       <mimic joint="${prefix}rightgear" multiplier="-1" offset="0"/>
     </joint>
+    <!-- Gazebo colors -->
+    <gazebo reference="${prefix}gripper_base">
+      <material>Gazebo/DarkGrey</material>
+    </gazebo>
+    <gazebo reference="${prefix}left_gear">
+      <material>Gazebo/DarkGrey</material>
+    </gazebo>
+    <gazebo reference="${prefix}right_gear">
+      <material>Gazebo/DarkGrey</material>
+    </gazebo>
+    <gazebo reference="${prefix}left_arm_bottom">
+      <material>Gazebo/DarkGrey</material>
+    </gazebo>
+    <gazebo reference="${prefix}right_arm_bottom">
+      <material>Gazebo/DarkGrey</material>
+    </gazebo>
+    <gazebo reference="${prefix}bottom_stick_left">
+      <material>Gazebo/DarkGrey</material>
+    </gazebo>
+    <gazebo reference="${prefix}bottom_stick_right">
+      <material>Gazebo/DarkGrey</material>
+    </gazebo>
+    <gazebo reference="${prefix}top_stick_left">
+      <material>Gazebo/DarkGrey</material>
+    </gazebo>
+    <gazebo reference="${prefix}top_stick_right">
+      <material>Gazebo/DarkGrey</material>
+    </gazebo>
+    <gazebo reference="${prefix}drive_gear">
+      <material>Gazebo/DarkGrey</material>
+    </gazebo>
     <!-- ros2_control -->
     <ros2_control name="${prefix}colman_gripper_system" type="system">

Commit message: fix wonky gripper behavior with mimic joints

File: src/gripper_description/gripper_description/urdf/colman-gripper.xacro (robot description, xacro)
@@ -1,4 +1,4 @@
 <robot xmlns:xacro="http://www.ros.org/wiki/xacro" name="colman-gripper">
-  <xacro:macro name="colman-gripper" params="prefix:='' visual_mesh_ext:='obj' include_gazebo_plugin:='true'">
+  <xacro:macro name="colman-gripper" params="prefix:='' visual_mesh_ext:='dae' include_gazebo_plugin:='true'">
     <xacro:property name="joint_limits_file" value="${xacro.load_yaml('$(find gripper_description)/config/joint_limits.yaml')}"/>
     <xacro:property name="joint_limits" value="${joint_limits_file['joint_limits']}"/>
@@ -289,34 +289,25 @@
     </joint>
     <!-- Gazebo colors -->
-    <gazebo reference="${prefix}gripper_base">
-      <material>Gazebo/DarkGrey</material>
-    </gazebo>
-    <gazebo reference="${prefix}left_gear">
-      <material>Gazebo/DarkGrey</material>
-    </gazebo>
-    <gazebo reference="${prefix}right_gear">
-      <material>Gazebo/DarkGrey</material>
-    </gazebo>
-    <gazebo reference="${prefix}left_arm_bottom">
-      <material>Gazebo/DarkGrey</material>
-    </gazebo>
-    <gazebo reference="${prefix}right_arm_bottom">
-      <material>Gazebo/DarkGrey</material>
-    </gazebo>
-    <gazebo reference="${prefix}bottom_stick_left">
-      <material>Gazebo/DarkGrey</material>
-    </gazebo>
-    <gazebo reference="${prefix}bottom_stick_right">
-      <material>Gazebo/DarkGrey</material>
-    </gazebo>
-    <gazebo reference="${prefix}top_stick_left">
-      <material>Gazebo/DarkGrey</material>
-    </gazebo>
-    <gazebo reference="${prefix}top_stick_right">
-      <material>Gazebo/DarkGrey</material>
-    </gazebo>
-    <gazebo reference="${prefix}drive_gear">
-      <material>Gazebo/DarkGrey</material>
-    </gazebo>
+    <xacro:macro name="gripper_material" params="link_name">
+      <gazebo reference="${link_name}">
+        <visual>
+          <material>
+            <ambient>0.2 0.2 0.2 1.0</ambient>
+            <diffuse>0.2 0.2 0.2 1.0</diffuse>
+            <specular>0.1 0.1 0.1 1.0</specular>
+          </material>
+        </visual>
+      </gazebo>
+    </xacro:macro>
+    <xacro:gripper_material link_name="${prefix}gripper_base"/>
+    <xacro:gripper_material link_name="${prefix}left_gear"/>
+    <xacro:gripper_material link_name="${prefix}right_gear"/>
+    <xacro:gripper_material link_name="${prefix}left_arm_bottom"/>
+    <xacro:gripper_material link_name="${prefix}right_arm_bottom"/>
+    <xacro:gripper_material link_name="${prefix}bottom_stick_left"/>
+    <xacro:gripper_material link_name="${prefix}bottom_stick_right"/>
+    <xacro:gripper_material link_name="${prefix}top_stick_left"/>
+    <xacro:gripper_material link_name="${prefix}top_stick_right"/>
+    <xacro:gripper_material link_name="${prefix}drive_gear"/>
     <!-- ros2_control -->
     <ros2_control name="${prefix}colman_gripper_system" type="system">
@@ -337,37 +328,4 @@
         <state_interface name="velocity"/>
       </joint>
-      <!-- Mimic joints -->
-      <joint name="${prefix}leftgear">
-        <state_interface name="position"/>
-        <state_interface name="velocity"/>
-      </joint>
-      <joint name="${prefix}rightgear">
-        <state_interface name="position"/>
-        <state_interface name="velocity"/>
-      </joint>
-      <joint name="${prefix}leftarm">
-        <state_interface name="position"/>
-        <state_interface name="velocity"/>
-      </joint>
-      <joint name="${prefix}rightarm">
-        <state_interface name="position"/>
-        <state_interface name="velocity"/>
-      </joint>
-      <joint name="${prefix}topleftstick">
-        <state_interface name="position"/>
-        <state_interface name="velocity"/>
-      </joint>
-      <joint name="${prefix}bottomleftstick">
-        <state_interface name="position"/>
-        <state_interface name="velocity"/>
-      </joint>
-      <joint name="${prefix}toprightstick">
-        <state_interface name="position"/>
-        <state_interface name="velocity"/>
-      </joint>
-      <joint name="${prefix}bottomrightstick">
-        <state_interface name="position"/>
-        <state_interface name="velocity"/>
-      </joint>
     </ros2_control>
     <!-- Gazebo ros2_control plugin -->
