Commit message: fix camera in moveit

File: src/oakd_description/oakd_description/urdf/oakd_pro.urdf.xacro (robot description, xacro)
@@ -13,5 +13,7 @@
                       <mesh filename="package://oakd_description/meshes/OAK-D-PRO.stl" />
               </geometry>
-               <material name="black" />
+               <material name="black">
+                 <color rgba="0.08 0.08 0.08 1.0" />
+               </material>
           </visual>
           <collision>

File: src/ur3e_moveit_config/config/ur3_robotiq.urdf.xacro (robot description, xacro)
@@ -1,6 +1,5 @@
 <?xml version="1.0"?>
 <robot xmlns:xacro="http://www.ros.org/wiki/xacro" name="ur3_robotiq">
-    <xacro:arg name="initial_positions_file" default="initial_positions.yaml" />
     <!-- Import ur3_robotiq urdf file -->
-    <xacro:include filename="$(find ros_robotiq_description)/urdf/moveit_urdf.urdf" />
+    <xacro:include filename="$(find ros_robotiq_description)/urdf/ur3e_robotiq.urdf.xacro" />
 </robot>

Commit message: fix camera urdf point cloud frame and rotation

File: src/oakd_description/oakd_description/urdf/oakd_pro.urdf.xacro (robot description, xacro)
@@ -31,6 +31,5 @@
       <!-- Add dummy joint for camera_optical_frame to link back to base_link -->
       <joint name="oakd_pro_camera_optical_joint_${mount_point}" type="fixed">
-      <!-- Point cloud frustrum is 90 degrees off from visual frame -->
-           <origin rpy="-1.57079632769 0 -1.570796332769" xyz="0 0 0" />
+           <origin rpy="0 0 3.14159265359" xyz="0 0 0" />
 	   <parent link="oakd_pro_${mount_point}" />
 	   <child link="oakd_pro_camera_optical_frame_${mount_point}" />
@@ -44,4 +43,10 @@
           </inertial>
   </link>
+  <joint name="oakd_pro_left_optical_joint_${mount_point}" type="fixed">
+    <origin xyz="-0.0375 0 0" rpy="0 0 0" />
+    <parent link="oakd_pro_camera_optical_frame_${mount_point}" />
+    <child link="oakd_pro_left_optical_frame_${mount_point}" />
+  </joint>
+  <link name="oakd_pro_left_optical_frame_${mount_point}" />
   <!-- Dummy joints for rgb camera to link back to base_link -->
         <joint name="oakd_pro_camera_rgb_optical_joint_${mount_point}" type="fixed">

Commit message: refactor ros_robotiq_description into smaller colman packages

File: src/oakd_description/oakd_description/urdf/oakd_pro.urdf.xacro (robot description, xacro)
@@ -1,156 +1,155 @@
-<?xml version="1.0" ?>
+<?xml version="1.0"?>
 <!--  xacro macros for oakd mount -->
-<robot name="oakd_pro" xmlns:xacro="http://ros.org/wiki/xacro">
-      <xacro:macro name="oakd_pro_link" params="mount_point">
-      <xacro:property name="oakd_pro_length" value="0.097" />
-      <xacro:property name="oakd_pro_width" value="0.0295" />
-      <xacro:property name="oakd_pro_depth" value="0.0229" />
-      <xacro:property name="oakd_pro_mass" value="0.091" />
-      <link name="oakd_pro_${mount_point}">
-          <visual>
-              <origin rpy="0 0 0" xyz="0 0 0" />
-              <geometry>
-                      <mesh filename="package://oakd_description/meshes/OAK-D-PRO.stl" />
-              </geometry>
-               <material name="black">
-                 <color rgba="0.08 0.08 0.08 1.0" />
-               </material>
-          </visual>
-          <collision>
-              <origin rpy="0 0 0" xyz="0 0 0" />
-              <geometry>
-                  <box size="${oakd_pro_length} ${oakd_pro_width} ${oakd_pro_depth}"/>
-              </geometry>
-          </collision>
-          <inertial>
-              <mass value="${oakd_pro_mass}" />
-              <origin xyz="0 0 0" rpy="0 0 0" />
-              <inertia ixx="0.0000105762" ixy="0.0" ixz="0.0" iyy="0.0000753284" iyz="0.0" izz="0.0000779510" />
-          </inertial>
-      </link>
-      <!-- Add dummy joint for camera_optical_frame to link back to base_link -->
-      <joint name="oakd_pro_camera_optical_joint_${mount_point}" type="fixed">
-           <origin rpy="0 0 3.14159265359" xyz="0 0 0" />
-	   <parent link="oakd_pro_${mount_point}" />
-	   <child link="oakd_pro_camera_optical_frame_${mount_point}" />
-	</joint>
-	<!-- Add dummy link for camera_optical_frame to link back to base_link -->
-        <link name="oakd_pro_camera_optical_frame_${mount_point}">
-        <inertial>
-	  <mass value="0.001" />
-	  <origin xyz="0 0 0" />
-	  <inertia ixx="0.0001" ixy="0.0" ixz="0.0" iyy="0.0001" iyz="0.0" izz="0.0001" />
-          </inertial>
-  </link>
-  <joint name="oakd_pro_left_optical_joint_${mount_point}" type="fixed">
-    <origin xyz="-0.0375 0 0" rpy="0 0 0" />
-    <parent link="oakd_pro_camera_optical_frame_${mount_point}" />
-    <child link="oakd_pro_left_optical_frame_${mount_point}" />
-  </joint>
-  <link name="oakd_pro_left_optical_frame_${mount_point}" />
-  <!-- Dummy joints for rgb camera to link back to base_link -->
-        <joint name="oakd_pro_camera_rgb_optical_joint_${mount_point}" type="fixed">
-           <origin rpy="-1.57079632679 0 -1.57079632679" xyz="0 0 0" />
-	   <parent link="oakd_pro_${mount_point}" />
-	   <child link="oakd_pro_camera_rgb_optical_frame_${mount_point}" />
-	</joint>
-	<!-- Add dummy link for camera_optical_frame to link back to base_link -->
-        <link name="oakd_pro_camera_rgb_optical_frame_${mount_point}">
-        <inertial>
-	  <mass value="0.001" />
-	  <origin xyz="0 0 0" />
-	  <inertia ixx="0.0001" ixy="0.0" ixz="0.0" iyy="0.0001" iyz="0.0" izz="0.0001" />
-          </inertial>
-  </link>
-  <!-- Harmonic sensors -->
-  <gazebo reference="oakd_pro_${mount_point}">
-    <material>Gazebo/DarkGrey</material>
-    <sensor name="oakd_pro_left_${mount_point}" type="camera">
-      <pose>0.0375 0 0 0 -1.5708 -1.5708</pose>
-      <always_on>true</always_on>
-      <topic>oakd_pro/left/image</topic>
-      <camera_info_topic>oakd_pro/left/camera_info</camera_info_topic>
-      <update_rate>30</update_rate>
-      <camera>
-        <horizontal_fov>1.3963</horizontal_fov>
-        <image>
-          <width>1280</width>
-          <height>800</height>
-          <format>L8</format>
-        </image>
-        <clip>
-          <near>0.3</near>
-          <far>35</far>
-        </clip>
-        <noise>
-          <type>gaussian</type>
-          <mean>0.0</mean>
-          <stddev>0.007</stddev>
-        </noise>
-      </camera>
-    </sensor>
-    <sensor name="oakd_pro_right_${mount_point}" type="camera">
-      <pose>-0.0375 0 0 0 -1.5708 -1.5708</pose>
-      <always_on>true</always_on>
-      <topic>oakd_pro/right/image</topic>
-      <camera_info_topic>oakd_pro/right/camera_info</camera_info_topic>
-      <update_rate>30</update_rate>
-      <camera>
-        <horizontal_fov>1.3963</horizontal_fov>
-        <image>
-          <width>1280</width>
-          <height>800</height>
-          <format>L8</format>
-        </image>
-        <clip>
-          <near>0.3</near>
-          <far>35</far>
-        </clip>
-        <noise>
-          <type>gaussian</type>
-          <mean>0.0</mean>
-          <stddev>0.007</stddev>
-        </noise>
-      </camera>
-    </sensor>
-    <sensor name="oakd_pro_rgb_${mount_point}" type="camera">
-      <pose>0 0 0 0 -1.5708 -1.5708</pose>
-      <always_on>true</always_on>
-      <topic>oakd_pro/rgb/image</topic>
-      <camera_info_topic>oakd_pro/rgb/camera_info</camera_info_topic>
-      <update_rate>30</update_rate>
-      <camera>
-        <horizontal_fov>1.1519</horizontal_fov>
-        <image>
-          <width>1920</width>
-          <height>1440</height>
-          <format>R8G8B8</format>
-        </image>
-        <clip>
-          <near>0.02</near>
-          <far>300</far>
-        </clip>
-        <noise>
-          <type>gaussian</type>
-          <mean>0.0</mean>
-          <stddev>0.007</stddev>
-        </noise>
-      </camera>
-    </sensor>
-  </gazebo>
-      <gazebo reference="oakd_pro_joint_${mount_point}">
-          <!-- <disableFixedJointLumping>true</disableFixedJointLumping>  -->
-          <!-- <preserveFixedJoint>true</preserveFixedJoint> -->
-      </gazebo>
-    </xacro:macro>
-    <xacro:macro name="oakd_pro_joint" params="x y z roll pitch yaw mount_point parent_link">
-        <joint name="oakd_pro_joint_${mount_point}" type="fixed">
-                <origin rpy="${roll} ${pitch} ${yaw}" xyz="${x} ${y} ${z}"/>
-            <parent link="${parent_link}" />
-            <child link="oakd_pro_${mount_point}" />
-        </joint>
-        <gazebo reference="oakd_pro_joint_${mount_point}">
-            <preserveFixedJoint>true</preserveFixedJoint>
-        </gazebo>
-    </xacro:macro>
+<robot xmlns:xacro="http://ros.org/wiki/xacro" name="oakd_pro">
+  <xacro:macro name="oakd_pro_link" params="mount_point">
+    <xacro:property name="oakd_pro_length" value="0.097"/>
+    <xacro:property name="oakd_pro_width" value="0.0295"/>
+    <xacro:property name="oakd_pro_depth" value="0.0229"/>
+    <xacro:property name="oakd_pro_mass" value="0.091"/>
+    <link name="oakd_pro_${mount_point}">
+      <visual>
+        <origin rpy="${pi/2} 0 0" xyz="0 0 0"/>
+        <geometry>
+          <mesh filename="package://oakd_description/meshes/OAK-D-PRO.obj"/>
+        </geometry>
+        <material name="black">
+          <color rgba="0.08 0.08 0.08 1.0"/>
+        </material>
+      </visual>
+      <collision>
+        <origin rpy="0 0 0" xyz="0 0 0"/>
+        <geometry>
+          <box size="${oakd_pro_length} ${oakd_pro_width} ${oakd_pro_depth}"/>
+        </geometry>
+      </collision>
+      <inertial>
+        <mass value="${oakd_pro_mass}"/>
+        <origin xyz="0 0 0" rpy="0 0 0"/>
+        <inertia ixx="0.0000105762" ixy="0.0" ixz="0.0" iyy="0.0000753284" iyz="0.0" izz="0.0000779510"/>
+      </inertial>
+    </link>
+    <!-- Add dummy joint for camera_optical_frame to link back to base_link -->
+    <joint name="oakd_pro_camera_optical_joint_${mount_point}" type="fixed">
+      <origin rpy="0 0 ${pi}" xyz="0 0 0"/>
+      <parent link="oakd_pro_${mount_point}"/>
+      <child link="oakd_pro_camera_optical_frame_${mount_point}"/>
+    </joint>
+    <!-- Add dummy link for camera_optical_frame to link back to base_link -->
+    <link name="oakd_pro_camera_optical_frame_${mount_point}">
+      <inertial>
+        <mass value="0.001"/>
+        <origin xyz="0 0 0"/>
+        <inertia ixx="0.0001" ixy="0.0" ixz="0.0" iyy="0.0001" iyz="0.0" izz="0.0001"/>
+      </inertial>
+    </link>
+    <joint name="oakd_pro_left_optical_joint_${mount_point}" type="fixed">
+      <origin xyz="-0.0375 0 0" rpy="0 0 0"/>
+      <parent link="oakd_pro_camera_optical_frame_${mount_point}"/>
+      <child link="oakd_pro_left_optical_frame_${mount_point}"/>
+    </joint>
+    <link name="oakd_pro_left_optical_frame_${mount_point}"/>
+    <!-- Dummy joints for rgb camera to link back to base_link -->
+    <joint name="oakd_pro_camera_rgb_optical_joint_${mount_point}" type="fixed">
+      <origin rpy="${-pi/2} 0 ${-pi/2}" xyz="0 0 0"/>
+      <parent link="oakd_pro_${mount_point}"/>
+      <child link="oakd_pro_camera_rgb_optical_frame_${mount_point}"/>
+    </joint>
+    <!-- Add dummy link for camera_optical_frame to link back to base_link -->
+    <link name="oakd_pro_camera_rgb_optical_frame_${mount_point}">
+      <inertial>
+        <mass value="0.001"/>
+        <origin xyz="0 0 0"/>
+        <inertia ixx="0.0001" ixy="0.0" ixz="0.0" iyy="0.0001" iyz="0.0" izz="0.0001"/>
+      </inertial>
+    </link>
+    <!-- Gazebo sensors -->
+    <gazebo reference="oakd_pro_${mount_point}">
+      <sensor name="oakd_pro_left_${mount_point}" type="camera">
+        <pose>0.0375 0 0 0 ${-pi/2} ${-pi/2}</pose>
+        <always_on>true</always_on>
+        <topic>oakd_pro/left/image</topic>
+        <camera_info_topic>oakd_pro/left/camera_info</camera_info_topic>
+        <update_rate>30</update_rate>
+        <camera>
+          <horizontal_fov>1.3963</horizontal_fov>
+          <image>
+            <width>1280</width>
+            <height>800</height>
+            <format>L8</format>
+          </image>
+          <clip>
+            <near>0.3</near>
+            <far>35</far>
+          </clip>
+          <noise>
+            <type>gaussian</type>
+            <mean>0.0</mean>
+            <stddev>0.007</stddev>
+          </noise>
+        </camera>
+      </sensor>
+      <sensor name="oakd_pro_right_${mount_point}" type="camera">
+        <pose>-0.0375 0 0 0 ${-pi/2} ${-pi/2}</pose>
+        <always_on>true</always_on>
+        <topic>oakd_pro/right/image</topic>
+        <camera_info_topic>oakd_pro/right/camera_info</camera_info_topic>
+        <update_rate>30</update_rate>
+        <camera>
+          <horizontal_fov>1.3963</horizontal_fov>
+          <image>
+            <width>1280</width>
+            <height>800</height>
+            <format>L8</format>
+          </image>
+          <clip>
+            <near>0.3</near>
+            <far>35</far>
+          </clip>
+          <noise>
+            <type>gaussian</type>
+            <mean>0.0</mean>
+            <stddev>0.007</stddev>
+          </noise>
+        </camera>
+      </sensor>
+      <sensor name="oakd_pro_rgb_${mount_point}" type="camera">
+        <pose>0 0 0 0 ${-pi/2} ${-pi/2}</pose>
+        <always_on>true</always_on>
+        <topic>oakd_pro/rgb/image</topic>
+        <camera_info_topic>oakd_pro/rgb/camera_info</camera_info_topic>
+        <update_rate>30</update_rate>
+        <camera>
+          <horizontal_fov>1.1519</horizontal_fov>
+          <image>
+            <width>1920</width>
+            <height>1440</height>
+            <format>R8G8B8</format>
+          </image>
+          <clip>
+            <near>0.02</near>
+            <far>300</far>
+          </clip>
+          <noise>
+            <type>gaussian</type>
+            <mean>0.0</mean>
+            <stddev>0.007</stddev>
+          </noise>
+        </camera>
+      </sensor>
+    </gazebo>
+    <gazebo reference="oakd_pro_joint_${mount_point}">
+      <!-- <disableFixedJointLumping>true</disableFixedJointLumping>  -->
+      <!-- <preserveFixedJoint>true</preserveFixedJoint> -->
+    </gazebo>
+  </xacro:macro>
+  <xacro:macro name="oakd_pro_joint" params="x y z roll pitch yaw mount_point parent_link">
+    <joint name="oakd_pro_joint_${mount_point}" type="fixed">
+      <origin rpy="${roll} ${pitch} ${yaw}" xyz="${x} ${y} ${z}"/>
+      <parent link="${parent_link}"/>
+      <child link="oakd_pro_${mount_point}"/>
+    </joint>
+    <gazebo reference="oakd_pro_joint_${mount_point}">
+      <preserveFixedJoint>true</preserveFixedJoint>
+    </gazebo>
+  </xacro:macro>
 </robot>
