Commit message: Model the custom gripper and limit shoulder pan to under a full turn
The arm has the custom gripper on it, not the vacuum. Default
gripper_type to custom, add a gripper_tip_link between the fingertips,
and make the link MoveIt targets a tip_link parameter set from
gripper_type instead of hardcoding vacuum_tip_link.

Limit shoulder_pan_joint to -270..+45 degrees so the arm can't wind its
cables around the base, and start sim/mock at -180 (facing the table) so
they begin inside the limits. Store Look3 as -pi rather than pi, the same
direction but inside the new limits.

File: src/colman_description/colman_description/urdf/colman.urdf.xacro (robot description, xacro)
@@ -56,5 +56,5 @@
   <xacro:arg name="use_mock_hardware" default="false"/>
   <xacro:arg name="mock_sensor_commands" default="false"/>
-  <xacro:arg name="initial_positions_file" default="$(find ur_description)/config/initial_positions.yaml"/>
+  <xacro:arg name="initial_positions_file" default="$(find colman_description)/config/initial_positions.yaml"/>
   <xacro:property name="initial_positions_file" value="$(arg initial_positions_file)"/>
   <!-- decide which link to attach the gripper to -->
@@ -74,4 +74,11 @@
       <child link="$(arg prefix)gripper_base"/>
       <origin xyz="0 0 ${'0.02' if '$(arg use_camera)' == 'true' else '0'}" rpy="${pi/2} 0 0"/>
+    </joint>
+    <!-- point between the fingertips, oriented like tool0 -->
+    <link name="$(arg prefix)gripper_tip_link"/>
+    <joint name="$(arg prefix)gripper_tip_joint" type="fixed">
+      <parent link="$(arg prefix)gripper_base"/>
+      <child link="$(arg prefix)gripper_tip_link"/>
+      <origin xyz="0 0.2 0" rpy="${-pi/2} 0 0"/>
     </joint>
   </xacro:if>

File: src/colman_gazebo/colman_gazebo/urdf/colman_gazebo.xacro (robot description, xacro)
@@ -7,5 +7,5 @@
   <!-- Gazebo specific args -->
   <xacro:arg name="mock_sensor_commands" default="false"/>
-  <xacro:arg name="initial_positions_file" default="$(find ur_description)/config/initial_positions.yaml"/>
+  <xacro:arg name="initial_positions_file" default="$(find colman_description)/config/initial_positions.yaml"/>
   <xacro:property name="initial_positions_file" default="$(arg initial_positions_file)"/>
   <!-- Gripper visuals and hardware interface -->

File: src/colman_moveit_config/srdf/arm.srdf.xacro (robot description, xacro)
@@ -39,5 +39,5 @@
         <joint name="elbow_joint" value="-0.6769"/>
         <joint name="shoulder_lift_joint" value="-1.4927"/>
-        <joint name="shoulder_pan_joint" value="${pi}"/>
+        <joint name="shoulder_pan_joint" value="${-pi}"/>
         <joint name="wrist_1_joint" value="-2.3952"/>
         <joint name="wrist_2_joint" value="1.6315"/>
